File: STEP-UP.sch (KiCad schematic (older format))
At the start: 7 parts, among them U3 MIC2251

Commit message: resolviendo error del componente AP9101CK6
Parts:
- C4: Mfg Part # (none) -> GRM21BR61E106KA73L
- C5: footprint Capacitor_SMD:C_0805_2012Metric -> Capacitor_SMD:C_0603_1608Metric; Mfg Part # (none) -> CL10B472KB8NNNC
- L1: Mfg Part # (none) -> SDR0403-100ML
- R5: Mfg Part # (none) -> RC0603FR-07100KL
- R6: Mfg Part # (none) -> RC0603FR-0733KL
Changed lines of the file:
@@
 F 2 "Capacitor_SMD:C_0805_2012Metric" H 4588 3800 50  0001 C CNN
 F 3 "~" H 4550 3950 50  0001 C CNN
+F 4 "GRM21BR61E106KA73L" H 4550 3950 50  0001 C CNN "Mfg Part #"
 	1    4550 3950
 	1    0    0    -1
@@
 F 2 "MSS_Devices:L_Bourns_SDR0403" H 5200 3150 50  0001 C CNN
 F 3 "~" H 5200 3150 50  0001 C CNN
+F 4 "SDR0403-100ML" H 5200 3150 50  0001 C CNN "Mfg Part #"
 	1    5200 3150
 	0    -1   -1   0
@@
 F 0 "C5" H 6865 3996 50  0000 L CNN
 F 1 "4.7nF" H 6865 3905 50  0000 L CNN
-F 2 "Capacitor_SMD:C_0805_2012Metric" H 6788 3800 50  0001 C CNN
+F 2 "Capacitor_SMD:C_0603_1608Metric" H 6788 3800 50  0001 C CNN
 F 3 "~" H 6750 3950 50  0001 C CNN
+F 4 "CL10B472KB8NNNC" H 6750 3950 50  0001 C CNN "Mfg Part #"
 	1    6750 3950
 	1    0    0    -1
@@
 F 2 "Resistor_SMD:R_0603_1608Metric" V 6180 3750 50  0001 C CNN
 F 3 "~" H 6250 3750 50  0001 C CNN
+F 4 "RC0603FR-07100KL" H 6250 3750 50  0001 C CNN "Mfg Part #"
 	1    6250 3750
 	-1   0    0    -1
@@
 F 2 "Resistor_SMD:R_0603_1608Metric" V 6180 4150 50  0001 C CNN
 F 3 "~" H 6250 4150 50  0001 C CNN
+F 4 "RC0603FR-0733KL" H 6250 4150 50  0001 C CNN "Mfg Part #"
 	1    6250 4150
 	-1   0    0    -1

Commit message: pasado a kicad 6
Parts:
- U3: symbol MSS_SourceSwitch:MIC2251 -> cargadorDeBateriasLitIon-rescue:MIC2251-MSS_SourceSwitch
Changed lines of the file:
@@
 $EndDescr
 $Comp
-L MSS_SourceSwitch:MIC2251 U?
+L cargadorDeBateriasLitIon-rescue:MIC2251-MSS_SourceSwitch U?
 U 1 1 5FB39CA8
 P 5200 3700
