File: cargadorDeBateriasLitIon.sch (KiCad schematic (older format))
At the start: 13 parts, among them Q1 2N7002, Q2 2N7002, U1 MCP73831-2, U2 AP9101C

Commit message: PCB version 1, falta probar
Parts:
- added J1: IN+, TestPoint:TestPoint_THTPad_1.5x1.5mm_Drill0.7mm, symbol Connector:Conn_01x01_Female
- added J2: IN-, TestPoint:TestPoint_THTPad_1.5x1.5mm_Drill0.7mm, symbol Connector:Conn_01x01_Female
- added J3: OUT+, TestPoint:TestPoint_THTPad_1.5x1.5mm_Drill0.7mm, symbol Connector:Conn_01x01_Female
- added J4: B+, TestPoint:TestPoint_THTPad_1.5x1.5mm_Drill0.7mm, symbol Connector:Conn_01x01_Female
- added J5: B-, TestPoint:TestPoint_THTPad_1.5x1.5mm_Drill0.7mm, symbol Connector:Conn_01x01_Female
- added J6: OUT-, TestPoint:TestPoint_THTPad_1.5x1.5mm_Drill0.7mm, symbol Connector:Conn_01x01_Female
Connections:
- wire segments 40 -> 44
Changed lines of the file:
@@
 encoding utf-8
 Sheet 1 1
-Title ""
-Date ""
-Rev ""
-Comp ""
+Title "Cargador de Baterias Litio"
+Date "2020-09-01"
+Rev "V 1.0.0"
+Comp "maykolrey.com"
 Comment1 ""
 Comment2 ""
@@
 Connection ~ 8450 3650
 Wire Wire Line
-	8450 3650 8700 3650
+	8450 3650 8800 3650
 Text Label 8700 3650 2    50   ~ 0
 B+
 Wire Wire Line
-	8450 3100 8700 3100
+	8450 3100 8800 3100
 Text Label 8700 3100 2    50   ~ 0
 OUT+
@@
 $EndComp
 Wire Wire Line
-	7700 4600 8700 4600
+	7700 4600 8800 4600
 Wire Wire Line
 	5300 3900 5300 4000
@@
 Wire Wire Line
 	3400 3600 3400 3500
-Wire Wire Line
-	3400 3100 3150 3100
 Connection ~ 3400 3100
 Text Label 3150 3100 0    50   ~ 0
@@
 	0    -1   1    0
 $EndComp
+$Comp
+L Connector:Conn_01x01_Female J1
+U 1 1 5F4DAD06
+P 2850 3100
+F 0 "J1" H 2742 2875 50  0000 C CNN
+F 1 "IN+" H 2742 2966 50  0000 C CNN
+F 2 "TestPoint:TestPoint_THTPad_1.5x1.5mm_Drill0.7mm" H 2850 3100 50  0001 C CNN
+F 3 "~" H 2850 3100 50  0001 C CNN
+	1    2850 3100
+	-1   0    0    1
+$EndComp
+Wire Wire Line
+	3050 3100 3400 3100
+$Comp
+L Connector:Conn_01x01_Female J3
+U 1 1 5F4DC6C5
+P 9000 3100
+F 0 "J3" H 9028 3126 50  0000 L CNN
+F 1 "OUT+" H 9028 3035 50  0000 L CNN
+F 2 "TestPoint:TestPoint_THTPad_1.5x1.5mm_Drill0.7mm" H 9000 3100 50  0001 C CNN
+F 3 "~" H 9000 3100 50  0001 C CNN
+	1    9000 3100
+	1    0    0    -1
+$EndComp
+$Comp
+L Connector:Conn_01x01_Female J4
+U 1 1 5F4DE4D2
+P 9000 3650
+F 0 "J4" H 9028 3676 50  0000 L CNN
+F 1 "B+" H 9028 3585 50  0000 L CNN
+F 2 "TestPoint:TestPoint_THTPad_1.5x1.5mm_Drill0.7mm" H 9000 3650 50  0001 C CNN
+F 3 "~" H 9000 3650 50  0001 C CNN
+	1    9000 3650
+	1    0    0    -1
+$EndComp
+$Comp
+L Connector:Conn_01x01_Female J5
+U 1 1 5F4DF38D
+P 9000 4600
+F 0 "J5" H 9028 4626 50  0000 L CNN
+F 1 "B-" H 9028 4535 50  0000 L CNN
+F 2 "TestPoint:TestPoint_THTPad_1.5x1.5mm_Drill0.7mm" H 9000 4600 50  0001 C CNN
+F 3 "~" H 9000 4600 50  0001 C CNN
+	1    9000 4600
+	1    0    0    -1
+$EndComp
+$Comp
+L Connector:Conn_01x01_Female J6
+U 1 1 5F4E06D9
+P 9000 4900
+F 0 "J6" H 9028 4926 50  0000 L CNN
+F 1 "OUT-" H 9028 4835 50  0000 L CNN
+F 2 "TestPoint:TestPoint_THTPad_1.5x1.5mm_Drill0.7mm" H 9000 4900 50  0001 C CNN
+F 3 "~" H 9000 4900 50  0001 C CNN
+	1    9000 4900
+	1    0    0    -1
+$EndComp
+$Comp
+L power:GND #PWR02
+U 1 1 5F4E0EDC
+P 8450 5100
+F 0 "#PWR02" H 8450 4850 50  0001 C CNN
+F 1 "GND" H 8455 4927 50  0000 C CNN
+F 2 "" H 8450 5100 50  0001 C CNN
+F 3 "" H 8450 5100 50  0001 C CNN
+	1    8450 5100
+	1    0    0    -1
+$EndComp
+Wire Wire Line
+	8450 5100 8450 4900
+Wire Wire Line
+	8450 4900 8800 4900
+$Comp
+L Connector:Conn_01x01_Female J2
+U 1 1 5F4E3B16
+P 2850 4900
+F 0 "J2" H 2742 5085 50  0000 C CNN
+F 1 "IN-" H 2742 4994 50  0000 C CNN
+F 2 "TestPoint:TestPoint_THTPad_1.5x1.5mm_Drill0.7mm" H 2850 4900 50  0001 C CNN
+F 3 "~" H 2850 4900 50  0001 C CNN
+	1    2850 4900
+	-1   0    0    -1
+$EndComp
+$Comp
+L power:GND #PWR01
+U 1 1 5F4E3B1C
+P 3400 5100
+F 0 "#PWR01" H 3400 4850 50  0001 C CNN
+F 1 "GND" H 3405 4927 50  0000 C CNN
+F 2 "" H 3400 5100 50  0001 C CNN
+F 3 "" H 3400 5100 50  0001 C CNN
+	1    3400 5100
+	-1   0    0    -1
+$EndComp
+Wire Wire Line
+	3400 5100 3400 4900
+Wire Wire Line
+	3400 4900 3050 4900
 $EndSCHEMATC

Commit message: generando gerber, faltan optimizar mas las pistas
Parts:
- removed Q1, Q2: 2N7002, Package_TO_SOT_SMD:SOT-23, symbol Device:Q_NMOS_GSD
- added Q1: FDC6401N, Package_TO_SOT_SMD:SuperSOT-6, symbol Mss_devices:FDC6401N
- U1: value MCP73831-2 -> MCP73831
- U2: value AP9101C -> AP9101CK6; footprint MSS_Devices:SOT25 -> MSS_Devices:SOT26; symbol Mss_devices:AP9101C -> Mss_devices:AP9101CK6; Mfg Part # AP9101CAK-AKTRG1 -> AP9101CK6-ADTRG1
Changed lines of the file:
@@
 P 4650 3500
 F 0 "U1" H 4650 4165 50  0000 C CNN
-F 1 "MCP73831-2" H 4650 4074 50  0000 C CNN
+F 1 "MCP73831" H 4650 4074 50  0000 C CNN
 F 2 "Package_TO_SOT_SMD:SOT-23-5" H 4650 3500 50  0001 C CNN
 F 3 "https://ww1.microchip.com/downloads/en/DeviceDoc/MCP73831-Family-Data-Sheet-DS20001984H.pdf" H 4650 3500 50  0001 C CNN
@@
 $EndComp
 $Comp
-L Mss_devices:AP9101C U2
+L Mss_devices:AP9101CK6 U2
 U 1 1 5F4AB55B
 P 6750 3750
 F 0 "U2" H 6750 4215 50  0000 C CNN
-F 1 "AP9101C" H 6750 4124 50  0000 C CNN
-F 2 "MSS_Devices:SOT25" H 7000 3750 50  0001 C CNN
+F 1 "AP9101CK6" H 6750 4124 50  0000 C CNN
+F 2 "MSS_Devices:SOT26" H 7000 3750 50  0001 C CNN
 F 3 "https://www.diodes.com/assets/Datasheets/AP9101C.pdf" H 7000 3750 50  0001 C CNN
-F 4 "AP9101CAK-AKTRG1" H 6750 3750 50  0001 C CNN "Mfg Part #"
+F 4 "AP9101CK6-ADTRG1" H 6750 3750 50  0001 C CNN "Mfg Part #"
 	1    6750 3750
 	-1   0    0    -1
@@
 	-1   0    0    -1
 $EndComp
-$Comp
-L Device:Q_NMOS_GSD Q1
-U 1 1 5F4AE73B
-P 6500 4500
-F 0 "Q1" V 6749 4500 50  0000 C CNN
-F 1 "2N7002" V 6840 4500 50  0000 C CNN
-F 2 "Package_TO_SOT_SMD:SOT-23" H 6700 4600 50  0001 C CNN
-F 3 "~" H 6500 4500 50  0001 C CNN
-F 4 "2N7002" H 6500 4500 50  0001 C CNN "Mfg Part #"
-	1    6500 4500
-	0    -1   1    0
-$EndComp
 Wire Wire Line
 	7000 4150 7000 4300
@@
 Connection ~ 8450 3100
 $Comp
-L Device:Q_NMOS_GSD Q2
-U 1 1 5F4D645C
-P 7000 4500
-F 0 "Q2" V 7249 4500 50  0000 C CNN
-F 1 "2N7002" V 7340 4500 50  0000 C CNN
-F 2 "Package_TO_SOT_SMD:SOT-23" H 7200 4600 50  0001 C CNN
-F 3 "~" H 7000 4500 50  0001 C CNN
-F 4 "2N7002" H 7000 4500 50  0001 C CNN "Mfg Part #"
-	1    7000 4500
-	0    -1   1    0
-$EndComp
-$Comp
 L Connector:Conn_01x01_Female J1
 U 1 1 5F4DAD06
@@
 Wire Wire Line
 	3400 4900 3050 4900
+$Comp
+L Mss_devices:FDC6401N Q1
+U 1 1 5F52AED7
+P 7000 4500
+F 0 "Q1" V 7249 4500 50  0000 C CNN
+F 1 "FDC6401N" V 7340 4500 50  0000 C CNN
+F 2 "Package_TO_SOT_SMD:SuperSOT-6" H 7200 4600 50  0001 C CNN
+F 3 "https://datasheet.lcsc.com/szlcsc/ON-Semicon-ON-FDC6401N_C154559.pdf" H 7000 4500 50  0001 C CNN
+	1    7000 4500
+	0    1    1    0
+$EndComp
+$Comp
+L Mss_devices:FDC6401N Q1
+U 2 1 5F52C56E
+P 6500 4500
+F 0 "Q1" V 6749 4500 50  0000 C CNN
+F 1 "FDC6401N" V 6840 4500 50  0000 C CNN
+F 2 "Package_TO_SOT_SMD:SuperSOT-6" H 6700 4600 50  0001 C CNN
+F 3 "https://datasheet.lcsc.com/szlcsc/ON-Semicon-ON-FDC6401N_C154559.pdf" H 6500 4500 50  0001 C CNN
+	2    6500 4500
+	0    1    1    0
+$EndComp
 $EndSCHEMATC

Commit message: agregando fuente de voltaje constante a 5V
Parts:
- removed C4: 100nF, Capacitor_SMD:C_0603_1608Metric, symbol Device:C
- J1, J2, J3, J4, J5, J6: Mfg Part # (none) -> DNP
- Q1: symbol Mss_devices:FDC6401N -> MSS_Transistor:FDC6401N; Mfg Part # (none) -> FDC6401N
- U1: symbol Mss_devices:MCP73831-2 -> Battery_Management:MCP73831-2-OT
- U2: symbol Mss_devices:AP9101CK6 -> Mss_devices:AP9101C
Connections:
- net labels added: VDD
- wire segments 44 -> 46
Other:
- moved on the sheet: C1, C2, C3, D1, J1, J2, J3, J4, J5, J6, R1, R2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

Commit message: resolviendo error del componente AP9101CK6
Parts:
- U2: symbol Mss_devices:AP9101C -> Mss_devices:AP9101C_SOT-26
Connections:
- net B-: now also U2.6 (VSS); no longer U2.3 (VSS)
- net at U2.1 (DO): now also Q1.1 (G); no longer R3.1
- net at C3.1, R4.1: now also U2.5 (VDD); no longer U2.2 (VDD)
- net at U2.4 (NC): no longer Q1.1 (G)
- net at Q1.3 (G): now also U2.3 (CO); no longer U2.5 (CO)
- new net: R3.1, U2.2 (VM)
Changed lines of the file:
@@
 $EndComp
 $Comp
-L Mss_devices:AP9101C U2
+L Mss_devices:AP9101C_SOT-26 U2
 U 1 1 5F4AB55B
 P 5250 3550

Commit message: pasado a kicad 6
Parts:
- Q1: symbol MSS_Transistor:FDC6401N -> cargadorDeBateriasLitIon-rescue:FDC6401N-MSS_Transistor
- U1: symbol Battery_Management:MCP73831-2-OT -> cargadorDeBateriasLitIon-rescue:MCP73831-2-OT-Battery_Management
- U2: symbol Mss_devices:AP9101C_SOT-26 -> cargadorDeBateriasLitIon-rescue:AP9101C_SOT-26-Mss_devices
Changed lines of the file:
@@
 $EndDescr
 $Comp
-L Battery_Management:MCP73831-2-OT U1
+L cargadorDeBateriasLitIon-rescue:MCP73831-2-OT-Battery_Management U1
 U 1 1 5F4A97F6
 P 3100 3000
@@
 $EndComp
 $Comp
-L Mss_devices:AP9101C_SOT-26 U2
+L cargadorDeBateriasLitIon-rescue:AP9101C_SOT-26-Mss_devices U2
 U 1 1 5F4AB55B
 P 5250 3550
@@
 	2000 3700 1650 3700
 $Comp
-L MSS_Transistor:FDC6401N Q1
+L cargadorDeBateriasLitIon-rescue:FDC6401N-MSS_Transistor Q1
 U 2 1 5F52AED7
 P 5500 4450
@@
 $EndComp
 $Comp
-L MSS_Transistor:FDC6401N Q1
+L cargadorDeBateriasLitIon-rescue:FDC6401N-MSS_Transistor Q1
 U 1 1 5F52C56E
 P 5000 4450
